File: control_board.sch (EAGLE design)
At the start: 19 parts

Commit message: schematic update
Parts:
- removed C1: (no value), SparkFun-Capacitors:10UF-25V-20%(PTH)
- removed R1: 330, resistor:R-US_0207/7
- removed V1, V2: 74540N, 74ttl-din:74540N
Connections:
- removed net +UB: C1.+, R1.2
- removed net N$1: JP1.2, V11.Y8
- removed net N$10: JP1.12, V21.Y6
- removed net N$11: JP1.13, V21.Y5
- removed net N$12: JP1.14, V21.Y4
- removed net N$13: JP1.10, V21.Y8
- removed net N$2: JP1.3, V11.Y7
- removed net N$3: JP1.4, V11.Y6
- removed net N$4: JP1.5, V11.Y5
- removed net N$5: JP1.6, V11.Y4
- removed net N$6: JP1.7, V11.Y3
- removed net N$7: JP1.8, V11.Y2
- removed net N$8: JP1.9, V11.Y1
- removed net N$9: JP1.11, V21.Y7
- net GND: no longer C1.-, V11.!G1, V11.!G2, V21.!G1, V21.!G2, V21.A1, V21.A2, V21.A3
- net LEVEL_SHIFTER_POWER_PIN: no longer R1.1
- net N$15: now also JP1.10; no longer V21.A8
- net N$16: now also JP1.11; no longer V21.A7
- net N$17: now also JP1.12; no longer V21.A6
- net N$18: now also JP1.13; no longer V21.A5
- net N$19: now also JP1.2; no longer V11.A8
- net N$20: now also JP1.3; no longer V11.A7
- net N$21: now also JP1.4; no longer V11.A6
- net N$22: now also JP1.5; no longer V11.A5
- net N$23: now also JP1.6; no longer V11.A4
- net N$24: now also JP1.7; no longer V11.A3
- net N$25: now also JP1.8; no longer V11.A2
- net N$26: now also JP1.9; no longer V11.A1
- net N$28: now also JP1.14; no longer V21.A4
